Commit message: legs control

File: src/nao_description/urdf/naoV33_generated_urdf/naoGazebo.xacro (robot description, xacro)
@@ -75,5 +75,5 @@
             <robotSimType>gazebo_ros_control/DefaultRobotHWSim</robotSimType>
         </plugin>
-<!--        <plugin filename="libgazebo_ros_imu.so" name="gazebo_ros_imu_controller">
+<!--        <plugin filename="libgazebo_ros_imu.so" name="">
             <robotNamespace>/nao_dcm</robotNamespace>
             <topicName>imu_data</topicName>
@@ -90,5 +90,5 @@
         </plugin>
 -->
-<!--        <plugin name="gazebo_ros_imu_controller" filename="${imu_plugin}">
+<!--        <plugin name="gazebo_ros_imu_controller" filename="">
             <robotNamespace>/nao_dcm</robotNamespace>
             <topicName>imu_data</topicName>

File: src/nao_description/urdf/naoV40_generated_urdf/nao.urdf (robot description, URDF)
Before this commit: robot nao, 83 links, 82 joints
Joints:
- joint LFinger11: mimic joint=LHand multiplier=0.999899 offset=0 -> (none); type continuous -> fixed
- joint LFinger12: mimic joint=LHand multiplier=0.999899 offset=0 -> (none); type continuous -> fixed
- joint LFinger13: mimic joint=LHand multiplier=0.999899 offset=0 -> (none); type continuous -> fixed
- joint LFinger21: mimic joint=LHand multiplier=0.999899 offset=0 -> (none); type continuous -> fixed
- joint LFinger22: mimic joint=LHand multiplier=0.999899 offset=0 -> (none); type continuous -> fixed
- joint LFinger23: mimic joint=LHand multiplier=0.999899 offset=0 -> (none); type continuous -> fixed
- joint LThumb1: mimic joint=LHand multiplier=0.999899 offset=0 -> (none); type continuous -> fixed
- joint LThumb2: mimic joint=LHand multiplier=0.999899 offset=0 -> (none); type continuous -> fixed
- joint RFinger11: mimic joint=RHand multiplier=0.999899 offset=0 -> (none); type continuous -> fixed
- joint RFinger12: mimic joint=RHand multiplier=0.999899 offset=0 -> (none); type continuous -> fixed
- joint RFinger13: mimic joint=RHand multiplier=0.999899 offset=0 -> (none); type continuous -> fixed
- joint RFinger21: mimic joint=RHand multiplier=0.999899 offset=0 -> (none); type continuous -> fixed
- joint RFinger22: mimic joint=RHand multiplier=0.999899 offset=0 -> (none); type continuous -> fixed
- joint RFinger23: mimic joint=RHand multiplier=0.999899 offset=0 -> (none); type continuous -> fixed
- joint RHand: origin xyz=0.05775 0 -0.01213 rpy=0 0 0 -> xyz=0.05775 0 -0.01231 rpy=0 0 0
- joint RThumb1: mimic joint=RHand multiplier=0.999899 offset=0 -> (none); type continuous -> fixed
- joint RThumb2: mimic joint=RHand multiplier=0.999899 offset=0 -> (none); type continuous -> fixed

File: src/nao_description/urdf/naoV40_generated_urdf/naoGazebo.xacro (robot description, xacro)
@@ -241,5 +241,5 @@
         <mu2>0.5</mu2>
         <selfCollide>false</selfCollide>
-        <turnGravityOff>true</turnGravityOff>
+        <turnGravityOff>false</turnGravityOff>
     </gazebo>
     <gazebo reference="LFinger12_link">
@@ -247,5 +247,5 @@
         <mu2>0.5</mu2>
         <selfCollide>false</selfCollide>
-        <turnGravityOff>true</turnGravityOff>
+        <turnGravityOff>false</turnGravityOff>
     </gazebo>
     <gazebo reference="LFinger13_link">
@@ -253,5 +253,5 @@
         <mu2>0.5</mu2>
         <selfCollide>false</selfCollide>
-        <turnGravityOff>true</turnGravityOff>
+        <turnGravityOff>false</turnGravityOff>
     </gazebo>
     <gazebo reference="LFinger21_link">
@@ -259,5 +259,5 @@
         <mu2>0.5</mu2>
         <selfCollide>false</selfCollide>
-        <turnGravityOff>true</turnGravityOff>
+        <turnGravityOff>false</turnGravityOff>
     </gazebo>
     <gazebo reference="LFinger22_link">
@@ -265,5 +265,5 @@
         <mu2>0.5</mu2>
         <selfCollide>false</selfCollide>
-        <turnGravityOff>true</turnGravityOff>
+        <turnGravityOff>false</turnGravityOff>
     </gazebo>
     <gazebo reference="LFinger23_link">
@@ -271,5 +271,5 @@
         <mu2>0.5</mu2>
         <selfCollide>false</selfCollide>
-        <turnGravityOff>true</turnGravityOff>
+        <turnGravityOff>false</turnGravityOff>
     </gazebo>
     <gazebo reference="LThumb1_link">
@@ -277,5 +277,5 @@
         <mu2>0.5</mu2>
         <selfCollide>false</selfCollide>
-        <turnGravityOff>true</turnGravityOff>
+        <turnGravityOff>false</turnGravityOff>
     </gazebo>
     <gazebo reference="LThumb2_link">
@@ -283,5 +283,5 @@
         <mu2>0.5</mu2>
         <selfCollide>false</selfCollide>
-        <turnGravityOff>true</turnGravityOff>
+        <turnGravityOff>false</turnGravityOff>
     </gazebo>
     <gazebo reference="LPelvis">
@@ -367,5 +367,5 @@
         <mu2>0.5</mu2>
         <selfCollide>false</selfCollide>
-        <turnGravityOff>true</turnGravityOff>
+        <turnGravityOff>false</turnGravityOff>
     </gazebo>
     <gazebo reference="RFinger12_link">
@@ -373,5 +373,5 @@
         <mu2>0.5</mu2>
         <selfCollide>false</selfCollide>
-        <turnGravityOff>true</turnGravityOff>
+        <turnGravityOff>false</turnGravityOff>
     </gazebo>
     <gazebo reference="RFinger13_link">
@@ -379,5 +379,5 @@
         <mu2>0.5</mu2>
         <selfCollide>false</selfCollide>
-        <turnGravityOff>true</turnGravityOff>
+        <turnGravityOff>false</turnGravityOff>
     </gazebo>
     <gazebo reference="RFinger21_link">
@@ -385,5 +385,5 @@
         <mu2>0.5</mu2>
         <selfCollide>false</selfCollide>
-        <turnGravityOff>true</turnGravityOff>
+        <turnGravityOff>false</turnGravityOff>
     </gazebo>
     <gazebo reference="RFinger22_link">
@@ -391,5 +391,5 @@
         <mu2>0.5</mu2>
         <selfCollide>false</selfCollide>
-        <turnGravityOff>true</turnGravityOff>
+        <turnGravityOff>false</turnGravityOff>
     </gazebo>
     <gazebo reference="RFinger23_link">
@@ -397,5 +397,5 @@
         <mu2>0.5</mu2>
         <selfCollide>false</selfCollide>
-        <turnGravityOff>true</turnGravityOff>
+        <turnGravityOff>false</turnGravityOff>
     </gazebo>
     <gazebo reference="RThumb1_link">
@@ -403,5 +403,5 @@
         <mu2>0.5</mu2>
         <selfCollide>false</selfCollide>
-        <turnGravityOff>true</turnGravityOff>
+        <turnGravityOff>false</turnGravityOff>
     </gazebo>
     <gazebo reference="RThumb2_link">
@@ -409,5 +409,5 @@
         <mu2>0.5</mu2>
         <selfCollide>false</selfCollide>
-        <turnGravityOff>true</turnGravityOff>
+        <turnGravityOff>false</turnGravityOff>
     </gazebo>
 <!--

File: src/nao_description/urdf/naoV40_generated_urdf/nao_fingers.xacro (robot description, xacro)
@@ -11,10 +11,10 @@
 		<xacro:insert_visu_RFinger23_link/>
 	</link>
-	<joint name="RFinger23" type="continuous">
+	<joint name="RFinger23" type="fixed">
 		<parent link="RFinger22_link"/>
 		<child link="RFinger23_link"/>
 		<origin rpy="0 0 -0.999899" xyz="0.01436 0 0"/>
 		<axis xyz="0 0 1.0"/>
-		<mimic joint="RHand" multiplier="0.999899" offset="0"/>
+	<!--	<mimic joint="RHand" multiplier="0.999899" offset="0"/> -->
 	</joint>
 	<link name="RFinger13_link">
@@ -25,10 +25,10 @@
 		<xacro:insert_visu_RFinger13_link/>
 	</link>
-	<joint name="RFinger13" type="continuous">
+	<joint name="RFinger13" type="fixed">
 		<parent link="RFinger12_link"/>
 		<child link="RFinger13_link"/>
 		<origin rpy="0 0 -0.999899" xyz="0.01436 0 0"/>
 		<axis xyz="0 0 1.0"/>
-		<mimic joint="RHand" multiplier="0.999899" offset="0"/>
+	<!--	<mimic joint="RHand" multiplier="0.999899" offset="0"/>  -->
 	</joint>
 	<link name="RFinger12_link">
@@ -39,10 +39,10 @@
 		<xacro:insert_visu_RFinger12_link/>
 	</link>
-	<joint name="RFinger12" type="continuous">
+	<joint name="RFinger12" type="fixed">
 		<parent link="RFinger11_link"/>
 		<child link="RFinger12_link"/>
 		<origin rpy="0 0 -0.999899" xyz="0.01436 0 0"/>
 		<axis xyz="0 0 1.0"/>
-		<mimic joint="RHand" multiplier="0.999899" offset="0"/>
+	<!--	<mimic joint="RHand" multiplier="0.999899" offset="0"/> -->
 	</joint>
 	<link name="LFinger21_link">
@@ -53,10 +53,10 @@
 		<xacro:insert_visu_LFinger21_link/>
 	</link>
-	<joint name="LFinger21" type="continuous">
+	<joint name="LFinger21" type="fixed">
 		<parent link="l_wrist"/>
 		<child link="LFinger21_link"/>
 		<origin rpy="1.25539 0.976662 -0.264067" xyz="0.06907 -0.01157 -0.00304"/>
 		<axis xyz="0 0 1.0"/>
-		<mimic joint="LHand" multiplier="0.999899" offset="0"/>
+	<!--	<mimic joint="LHand" multiplier="0.999899" offset="0"/> -->
 	</joint>
 	<link name="LFinger13_link">
@@ -67,10 +67,10 @@
 		<xacro:insert_visu_LFinger13_link/>
 	</link>
-	<joint name="LFinger13" type="continuous">
+	<joint name="LFinger13" type="fixed">
 		<parent link="LFinger12_link"/>
 		<child link="LFinger13_link"/>
 		<origin rpy="0 0 -0.999899" xyz="0.01436 0 0"/>
 		<axis xyz="0 0 1.0"/>
-		<mimic joint="LHand" multiplier="0.999899" offset="0"/>
+	<!--	<mimic joint="LHand" multiplier="0.999899" offset="0"/> -->
 	</joint>
 	<link name="LFinger11_link">
@@ -81,10 +81,10 @@
 		<xacro:insert_visu_LFinger11_link/>
 	</link>
-	<joint name="LFinger11" type="continuous">
+	<joint name="LFinger11" type="fixed">
 		<parent link="l_wrist"/>
 		<child link="LFinger11_link"/>
 		<origin rpy="1.8862 0.976662 0.264067" xyz="0.06907 0.01157 -0.00304"/>
 		<axis xyz="0 0 1.0"/>
-		<mimic joint="LHand" multiplier="0.999899" offset="0"/>
+	<!--	<mimic joint="LHand" multiplier="0.999899" offset="0"/> -->
 	</joint>
 	<link name="RFinger22_link">
@@ -95,10 +95,10 @@
 		<xacro:insert_visu_RFinger22_link/>
 	</link>
-	<joint name="RFinger22" type="continuous">
+	<joint name="RFinger22" type="fixed">
 		<parent link="RFinger21_link"/>
 		<child link="RFinger22_link"/>
 		<origin rpy="0 0 -0.999899" xyz="0.01436 0 0"/>
 		<axis xyz="0 0 1.0"/>
-		<mimic joint="RHand" multiplier="0.999899" offset="0"/>
+	<!--	<mimic joint="RHand" multiplier="0.999899" offset="0"/> -->
 	</joint>
 	<link name="LFinger22_link">
@@ -109,10 +109,10 @@
 		<xacro:insert_visu_LFinger22_link/>
 	</link>
-	<joint name="LFinger22" type="continuous">
+	<joint name="LFinger22" type="fixed">
 		<parent link="LFinger21_link"/>
 		<child link="LFinger22_link"/>
 		<origin rpy="0 0 -0.999899" xyz="0.01436 0 0"/>
 		<axis xyz="0 0 1.0"/>
-		<mimic joint="LHand" multiplier="0.999899" offset="0"/>
+	<!--	<mimic joint="LHand" multiplier="0.999899" offset="0"/> -->
 	</joint>
 	<link name="RFinger21_link">
@@ -123,10 +123,10 @@
 		<xacro:insert_visu_RFinger21_link/>
 	</link>
-	<joint name="RFinger21" type="continuous">
+	<joint name="RFinger21" type="fixed">
 		<parent link="r_wrist"/>
 		<child link="RFinger21_link"/>
 		<origin rpy="1.25539 0.976662 -0.264067" xyz="0.06907 -0.01157 -0.00304"/>
 		<axis xyz="0 0 1.0"/>
-		<mimic joint="RHand" multiplier="0.999899" offset="0"/>
+	<!--	<mimic joint="RHand" multiplier="0.999899" offset="0"/> -->
 	</joint>
 	<link name="LFinger12_link">
@@ -137,10 +137,10 @@
 		<xacro:insert_visu_LFinger12_link/>
 	</link>
-	<joint name="LFinger12" type="continuous">
+	<joint name="LFinger12" type="fixed">
 		<parent link="LFinger11_link"/>
 		<child link="LFinger12_link"/>
 		<origin rpy="0 0 -0.999899" xyz="0.01436 0 0"/>
 		<axis xyz="0 0 1.0"/>
-		<mimic joint="LHand" multiplier="0.999899" offset="0"/>
+	<!--	<mimic joint="LHand" multiplier="0.999899" offset="0"/> -->
 	</joint>
 	<link name="RFinger11_link">
@@ -151,10 +151,10 @@
 		<xacro:insert_visu_RFinger11_link/>
 	</link>
-	<joint name="RFinger11" type="continuous">
+	<joint name="RFinger11" type="fixed">
 		<parent link="r_wrist"/>
 		<child link="RFinger11_link"/>
 		<origin rpy="1.8862 0.976662 0.264067" xyz="0.06907 0.01157 -0.00304"/>
 		<axis xyz="0 0 1.0"/>
-		<mimic joint="RHand" multiplier="0.999899" offset="0"/>
+	<!--	<mimic joint="RHand" multiplier="0.999899" offset="0"/> -->
 	</joint>
 	<link name="LFinger23_link">
@@ -165,24 +165,24 @@
 		<xacro:insert_visu_LFinger23_link/>
 	</link>
-	<joint name="LFinger23" type="continuous">
+	<joint name="LFinger23" type="fixed">
 		<parent link="LFinger22_link"/>
 		<child link="LFinger23_link"/>
 		<origin rpy="0 0 -0.999899" xyz="0.01436 0 0"/>
 		<axis xyz="0 0 1.0"/>
-		<mimic joint="LHand" multiplier="0.999899" offset="0"/>
+	<!--	<mimic joint="LHand" multiplier="0.999899" offset="0"/> -->
 	</joint>
 	<link name="LThumb1_link">
 		<inertial>
 			<mass value="2e-06"/>
-			<inertia ixx="1.1e-09" ixy="0" ixz="0" iyy="1.1e-09" iyz="0" izz="1.1e-09"/>
+			<inertia ixx="1.1e-09" ixy="0" ixz="0" iyy="0" iyz="0" izz="0"/>
 		</inertial>
 		<xacro:insert_visu_LThumb1_link/>
 	</link>
-	<joint name="LThumb1" type="continuous">
+	<joint name="LThumb1" type="fixed">
 		<parent link="l_wrist"/>
 		<child link="LThumb1_link"/>
 		<origin rpy="-1.5708 0.0472984 -3.26826e-08" xyz="0.04895 0 -0.02638"/>
 		<axis xyz="0 0 1.0"/>
-		<mimic joint="LHand" multiplier="0.999899" offset="0"/>
+	<!--	<mimic joint="LHand" multiplier="0.999899" offset="0"/> -->
 	</joint>
 	<link name="RThumb1_link">
@@ -193,38 +193,38 @@
 		<xacro:insert_visu_RThumb1_link/>
 	</link>
-	<joint name="RThumb1" type="continuous">
+	<joint name="RThumb1" type="fixed">
 		<parent link="r_wrist"/>
 		<child link="RThumb1_link"/>
 		<origin rpy="-1.5708 0.0472984 -3.26826e-08" xyz="0.04895 0 -0.02638"/>
 		<axis xyz="0 0 1.0"/>
-		<mimic joint="RHand" multiplier="0.999899" offset="0"/>
+	<!--	<mimic joint="RHand" multiplier="0.999899" offset="0"/> -->
 	</joint>
 	<link name="RThumb2_link">
 		<inertial>
 			<mass value="2e-06"/>
-			<inertia ixx="1.1e-09" ixy="0" ixz="0" iyy="1.1e-09" iyz="0" izz="1.1e-09"/>
+			<inertia ixx="0" ixy="0" ixz="0" iyy="0" iyz="0" izz="0"/>
 		</inertial>
 		<xacro:insert_visu_RThumb2_link/>
 	</link>
-	<joint name="RThumb2" type="continuous">
+	<joint name="RThumb2" type="fixed">
 		<parent link="RThumb1_link"/>
 		<child link="RThumb2_link"/>
 		<origin rpy="0 0 -0.999899" xyz="0.01436 0 0"/>
 		<axis xyz="0 0 1.0"/>
-		<mimic joint="RHand" multiplier="0.999899" offset="0"/>
+	<!--	<mimic joint="RHand" multiplier="0.999899" offset="0"/> -->
 	</joint>
 	<link name="LThumb2_link">
 		<inertial>
 			<mass value="2e-06"/>
-			<inertia ixx="1.1e-09" ixy="0" ixz="0" iyy="1.1e-09" iyz="0" izz="1.1e-09"/>
+			<inertia ixx="0" ixy="0" ixz="0" iyy="0" iyz="0" izz="0"/>
 		</inertial>
 		<xacro:insert_visu_LThumb2_link/>
 	</link>
-	<joint name="LThumb2" type="continuous">
+	<joint name="LThumb2" type="fixed">
 		<parent link="LThumb1_link"/>
 		<child link="LThumb2_link"/>
 		<origin rpy="0 0 -0.999899" xyz="0.01436 0 0"/>
 		<axis xyz="0 0 1.0"/>
-		<mimic joint="LHand" multiplier="0.999899" offset="0"/>
+	<!--	<mimic joint="LHand" multiplier="0.999899" offset="0"/> -->
 	</joint>
 </robot>
